File: hardware/USBSID-Pico-v1.0/USBSID-Pico-v1.0.kicad_pcb (KiCad board)
At the start: 2 copper layers, 92.8 x 71.8 mm, 95 parts, among them J1 SID1 (DIP28-Wide-socket), J10 BP, J11 GND/S1, J12 12v/9v, J13 A5, J14 UART, J15 BP, J16 S2/GND, J17 6581, J18 6581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

Commit message: Update v1.0 pcb with OSHWA certification
Parts:
- added REF**: OSHW_US1.0_-Certification-Mark-Stacked_8x7mm_SilkScreen, LouD:OSHW_US1.0_-Certification-Mark-Stacked_8x7mm_SilkScreen, B.Cu at (128.7, 63.2)
