File: hardware/USBSID-Pico-v1.0/USBSID-Pico-v1.0.kicad_sch (KiCad schematic)
At the start: 43 parts, among them J1 SID1 (DIP28-Wide-socket), J11 GND/S1, J16 S2/GND, J17 6581, J18 6581, J2 SID2 (DIP28-Wide-socket), J20 AudioJack2_Ground_Switch, J3 1MHz Crystal, J4 OSC EN, J5 S1 6581/8580 J1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

Commit message: Update v1.0 pcb with OSHWA certification
Parts:
- added LOGO1: ~, symbol OSHW_Certification_Mark:OSHW_US10_Certification_Mark_Wide_Medium
Changed lines of the file:
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@@
+		)
+	)
+	(symbol
+		(lib_id "OSHW_Certification_Mark:OSHW_US10_Certification_Mark_Wide_Medium")
+		(at 222.25 173.99 0)
+		(unit 1)
+		(exclude_from_sim no)
+		(in_bom no)
+		(on_board no)
+		(dnp no)
+		(fields_autoplaced yes)
+		(property "Reference" "LOGO1"
+			(at 222.25 173.99 0)
+			(effects
+				(font
+					(size 1.27 1.27)
+				)
+				(hide yes)
+			)
+		)
+		(property "Value" "~"
+			(at 222.25 173.99 0)
+			(effects
+				(font
+					(size 1.27 1.27)
+				)
+				(hide yes)
+			)
+		)
+		(property "Footprint" ""
+			(at 222.25 173.99 0)
+			(effects
+				(font
+					(size 1.27 1.27)
+				)
+				(hide yes)
+			)
+		)
+		(property "Datasheet" ""
+			(at 222.25 173.99 0)
+			(effects
+				(font
+					(size 1.27 1.27)
+				)
+				(hide yes)
+			)
+		)
+		(property "Description" "OSHW Certification Mark, Wide"
+			(at 222.25 173.99 0)
+			(effects
+				(font
+					(size 1.27 1.27)
+				)
+				(hide yes)
+			)
+		)
+		(instances
+			(project ""
+				(path "/f639dbf8-eb43-4301-9a54-898621165136"
+					(reference "LOGO1")
+					(unit 1)
+				)
+			)
 		)
 	)
