File: hardware/Volume-daughterboard/Volume-daughterboard.kicad_sch (KiCad schematic)
At the start: 32 parts, among them J1 GND/S1, J2 S2/GND, J4 1503 17, U1 OPA1688IDR

Commit message: Volume daughterboard
Parts:
- C1, C2: Manufacturer (none) -> FOJAN; Mfg Part # (none) -> FCC0805B104K500DT; Mfg Part Desc (none) -> CAP CER 100nF 50V X7R 0805
- C10, C9: Manufacturer (none) -> FOJAN; Mfg Part # (none) -> FCC0805B105K500FT; Mfg Part Desc (none) -> CAP CER 1uF 50V X7R 0805
- C11, C5, C6: Manufacturer (none) -> FOJAN; Mfg Part # (none) -> FCC0805X106K500FT; Mfg Part Desc (none) -> CAP CER 10uF 50V X5R 0805
- C3, C4: Manufacturer (none) -> FOSAN; Mfg Part # (none) -> FVH016ADA470M0554; Mfg Part Desc (none) -> CAP ALUM 47uF ±20% 16V SMD
- C7, C8: Manufacturer (none) -> FOJAN; Mfg Part # (none) -> FCC0805N101J500BT; Mfg Part Desc (none) -> CAP CER 100pF 50V C0G 0805
- D1: Mfg Part Desc BAT54C SOT-23 -> DIODE ARR SCHOTTKY 30V SOT-23
- J1, J2: Mfg Part Desc Through Hole Pin Header 2.5mm 6mm 3P -40℃~+105℃ 3mm 2.54mm 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 -> PH2.54-01-04PZD
- J4: Manufacturer (none) -> Lumberg; Mfg Part # (none) -> 134382 1503-17 / SJ1-3525N; Mfg Part Desc (none) -> Through Hole Audio Connectors RoHS
- R1, R2: Mfg Part Desc 125mW Thick Film Resistors 150V ±100ppm/℃ ±1% 10kΩ 0805 Chi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 -> RES 10kΩ ±1% 125mW 0805
- R10, R9: Mfg Part Desc (none) -> RES 10kΩ ±1% 125mW 0805
- R3, R4: Mfg Part # (none) -> 0805W8F100JT5E; Mfg Part Desc (none) -> RES 10Ω ±1% 125mW 0805
- R5, R6, R7, R8: Mfg Part # (none) -> 0805W8F4702T5E; Mfg Part Desc (none) -> RES 47kΩ ±1% 125mW 0805
- RV1, RV2: Manufacturer (none) -> ALPSALPINE; Mfg Part # (none) -> RK09K1130AAU; Mfg Part Desc (none) -> POT 10kΩ Through Hole
- U1: Mfg Part # OPA1688ID -> OPA1688IDR; Mfg Part Desc OPA1688 SOIC-8 -> 36-V, Single-Supply, 10-MHz, Rail-to-Rail Output Operationa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
